File: Hardware/pcb/xFaders/xfaders.sch (KiCad schematic (older format))
At the start: 27 parts, among them J1 Conn_01x03_Male, J10 Conn_01x03_Male, J11 Conn_01x03_Male, J12 Conn_01x03_Male, J13 Conn_01x03_Male, J14 Conn_01x03_Male, J15 Conn_01x03_Male, J16 Conn_02x10_Odd_Even, J17 Conn_02x10_Odd_Even, J18 Conn_02x10_Odd_Even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

Commit message: Update PCB for new RGB LEDs and 5V power supply
Parts:
- added C1, C2: 10 uF, Capacitor_SMD:C_0603_1608Metric_Pad1.05x0.95mm_HandSolder, symbol Device:CP_Small
- added J19: PWR In, Connector_PinHeader_2.54mm:PinHeader_1x02_P2.54mm_Vertical, symbol Connector:Screw_Terminal_01x02
- added J20, J21, J22: 5V, Connector_PinHeader_2.54mm:PinHeader_1x02_P2.54mm_Vertical, symbol Connector:Conn_01x02_Male
- added Q1: 2N7000, Package_TO_SOT_THT:TO-92_Inline, symbol Transistor_FET:2N7000
- added R7, R8: 10k, Resistor_THT:R_Axial_DIN0207_L6.3mm_D2.5mm_P7.62mm_Horizontal, symbol Device:R_Small
- added U4: LM1084-5.0, Package_TO_SOT_THT:TO-220-3_Vertical, symbol Regulator_Linear:LM1084-5.0
- R1, R2, R3, R4, R5, R6: footprint (none) -> Resistor_THT:R_Axial_DIN0207_L6.3mm_D2.5mm_P7.62mm_Horizontal
- U2: symbol bluepill_breakouts:BluePill_STM32F103C -> xfaders-rescue:BluePill_STM32F103C-bluepill_breakouts
Connections:
- net Vdd: now also Q1.2 (G), R7.1; no longer J16.1 (Pin_1), J17.1 (Pin_1), J18.1 (Pin_1)
- net at U1.10 (B), U3.10 (B): now also U2.27 (PA10_RX1); no longer U2.22 (PB13_SCK2)
- net SPI_3V3: now reaches U2.24 (PB15_MOSI2)
- net SPI_3V3: now also Q1.1 (S), R7.2
- net at J16.18 (Pin_18): now also J17.1 (Pin_1)
- net at J17.18 (Pin_18): now also J18.1 (Pin_1)
- net VEE renamed GND
- net GND: now also C1.2, C2.2, J19.1 (Pin_1), J20.1 (Pin_1), J21.1 (Pin_1), J22.1 (Pin_1), U4.1 (GND)
- new net: C1.1, J19.2 (Pin_2), U4.3 (VI)
- new net SPI_5V: J16.1 (Pin_1), Q1.3 (D), R8.2
- new net VCC5V: C2.1, J20.2 (Pin_2), J21.2 (Pin_2), J22.2 (Pin_2), R8.1, U4.2 (VO)
- no-connect marks 15 -> 12
Other:
- note added: "5V 5A power supply"
- note added: "SPI step-up converter"
- note added: "see: http://electronictoofree.blogspot.com/2018/04/reading-schematic-sparkfun.html"

Commit message: Add gerber files for version 2.0
Parts:
- C1, C2: footprint Capacitor_SMD:C_0603_1608Metric_Pad1.05x0.95mm_HandSolder -> Capacitor_THT:C_Disc_D5.0mm_W2.5mm_P5.00mm
Changed lines of the file:
@@
 F 0 "C2" H 2538 5996 50  0000 L CNN
 F 1 "10 uF" H 2538 5905 50  0000 L CNN
-F 2 "Capacitor_SMD:C_0603_1608Metric_Pad1.05x0.95mm_HandSolder" H 2450 5950 50  0001 C CNN
+F 2 "Capacitor_THT:C_Disc_D5.0mm_W2.5mm_P5.00mm" H 2450 5950 50  0001 C CNN
 F 3 "~" H 2450 5950 50  0001 C CNN
 	1    2450 5950
@@
 F 0 "C1" H 1488 5996 50  0000 L CNN
 F 1 "10 uF" H 1488 5905 50  0000 L CNN
-F 2 "Capacitor_SMD:C_0603_1608Metric_Pad1.05x0.95mm_HandSolder" H 1400 5950 50  0001 C CNN
+F 2 "Capacitor_THT:C_Disc_D5.0mm_W2.5mm_P5.00mm" H 1400 5950 50  0001 C CNN
 F 3 "~" H 1400 5950 50  0001 C CNN
 	1    1400 5950
